Commit message: Add real MoveIT Launch&Controllers + FakeHardwareTrue + SimIntact

File: ros2_ws/src/ur5e_cell_description/urdf/ur5e_cell.urdf.xacro (robot description, xacro)
@@ -5,6 +5,12 @@
   <!-- Vendor YAMLs (Humble layout) -->
   <xacro:arg name="ur_type"             default="ur5e"/>
+  <xacro:arg name="tf_prefix"           default=""/>
+  <xacro:arg name="parent"              default="world"/>
+  <xacro:arg name="name"                default="ur5e_cell"/>
   <xacro:arg name="kinematics_params"   default="$(find ur_description)/config/$(arg ur_type)/default_kinematics.yaml"/>
   <xacro:arg name="joint_limit_params"  default="$(find ur_description)/config/$(arg ur_type)/joint_limits.yaml"/>
+  <xacro:arg name="joint_limits_parameters_file" default="$(arg joint_limit_params)"/>
+  <xacro:property name="joint_limits_file"
+                  value="${joint_limits_parameters_file if joint_limits_parameters_file else joint_limit_params}"/>
   <xacro:arg name="physical_params"     default="$(find ur_description)/config/$(arg ur_type)/physical_parameters.yaml"/>
   <xacro:arg name="visual_params"       default="$(find ur_description)/config/$(arg ur_type)/visual_parameters.yaml"/>
@@ -13,11 +19,13 @@
   <!-- Instantiate our cell geometry (the vendor will inject ONE control block internally) -->
   <xacro:ur5e_cell
-      parent="world"
-      ur_type="$(arg ur_type)"
-      joint_limits_parameters_file="$(arg joint_limit_params)"
-      kinematics_parameters_file="$(arg kinematics_params)"
-      physical_parameters_file="$(arg physical_params)"
-      visual_parameters_file="$(arg visual_params)">
-    <origin xyz="0 0 0.9" rpy="0 0 0"/>
+    parent="$(arg parent)"
+    ur_type="$(arg ur_type)"
+    name="$(arg name)"
+    tf_prefix="$(arg tf_prefix)"
+    joint_limits_parameters_file="$(arg joint_limits_parameters_file)"
+    kinematics_parameters_file="$(arg kinematics_params)"
+    physical_parameters_file="$(arg physical_params)"
+    visual_parameters_file="$(arg visual_params)">
+    <origin xyz="0 0 0" rpy="0 0 0"/>
   </xacro:ur5e_cell>
   <!-- No <ros2_control> tag here. No vendor control include here. -->

File: ros2_ws/src/ur5e_cell_description/urdf/ur5e_cell_macro.xacro (robot description, xacro)
@@ -2,12 +2,6 @@
 <robot xmlns:xacro="http://www.ros.org/wiki/xacro">
   <xacro:include filename="$(find ur_description)/urdf/ur_macro.xacro"/>
-  <xacro:macro name="ur5e_cell" params="
-      parent
-      *origin
-      ur_type
-      joint_limits_parameters_file
-      kinematics_parameters_file
-      physical_parameters_file
-      visual_parameters_file">
+  <xacro:macro name="ur5e_cell" params="parent:='world' *origin ur_type name tf_prefix:='' kinematics_parameters_file joint_limits_parameters_file physical_parameters_file visual_parameters_file">
+    <xacro:property name="tool0_link_name" value="${tf_prefix + '_tool0' if tf_prefix else 'tool0'}"/>
     <joint name="pedestal_joint" type="fixed">
       <xacro:insert_block name="origin"/>
@@ -17,6 +11,6 @@
     <link name="pedestal"/>
     <xacro:ur_robot
-      name="${ur_type}"
-      tf_prefix="${ur_type}_"
+      name="${name}"
+      tf_prefix="${tf_prefix}"
       parent="pedestal"
       joint_limits_parameters_file="${joint_limits_parameters_file}"
@@ -45,5 +39,5 @@
     </link>
     <joint name="tool0_to_simple_gripper" type="fixed">
-      <parent link="${ur_type}_tool0"/>
+      <parent link="${tool0_link_name}"/>
       <child  link="simple_gripper"/>
       <origin xyz="0 0 0.08" rpy="0 0 0"/>
